Commit message: modifiche al file yaml

File: simple_example_description/urdf/robot.urdf (robot description, URDF)
Before this commit: robot simple_example, 2 links, 1 joints
Links:
- added link third_link, mass 0.10; collision box size=0.02 0.02 0.05; visual box size=0.02 0.02 0.05
Joints:
- added joint base_to_third_joint: type continuous, parent second_link, child third_link, origin xyz=0.0 0.0 0.1 rpy=0.0 0.0 0.0, axis 1 0 0
- joint base_to_second_joint: axis 1 0 0 -> 0 0 1
